File: kicad/hellerune.kicad_pcb (KiCad board)
At the start: 4 copper layers, 98.5 x 57 mm, 66 parts, among them IC1 CD4049UBE, J1 GND1, J10 SWITCHY-2-B-IN-R1, J11 9VOUT2, J12 GND4, J2 GND2, J3 GND3, J4 GND4, J5 Conn_01x02_Female, J6 9VIN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

Commit message: pcb draft complete
Parts:
- added C22: 10nF, Capacitor_SMD:C_0805_2012Metric, F.Cu at (146.4, 93.8)
- moved D3 27.5 mm to (151.3, 80.4)
- moved R23 13.6 mm to (140.6, 79.2), turned to 180 degrees
- moved C20 8.75 mm to (155.0, 89.0), turned to 90 degrees
- moved R15 7.60 mm to (147.7, 98.6), turned to 180 degrees
- moved C8 7.57 mm to (153.3, 105.4)
- moved R18 7.44 mm to (153.9, 98.4)
- moved C17 5.79 mm to (125.4, 77.4)
- moved C21 3.09 mm to (146.2, 82.0)
- moved U4 2.62 mm to (144.7, 86.5)
- moved R21 1.78 mm to (135.0, 82.4)
Connections:
- C13 pad 1: Net-(D3-K) -> CD-VCC
- C21 pad 1: Net-(D3-K) -> CD-VCC
- C8 pad 1: Net-(D3-K) -> CD-VCC
- D3 pad 1: Net-(D3-K) -> CD-VCC
- IC1 pad 1: VREF -> CD-VCC
- IC1 pad 11: VREF -> CD-VCC
- IC1 pad 5: VREF -> CD-VCC
- IC1 pad 7: VREF -> CD-VCC
- IC1 pad 9: VREF -> CD-VCC
- R15 pad 1: Net-(D3-K) -> CD-VCC
- U3 pad 8: Net-(D3-K) -> CD-VCC
- U4 pad 8: Net-(D3-K) -> CD-VCC
Routing:
- net CD-VCC: track 0.00 -> 125.8 mm, vias 0 -> 4
- net Net-(U4B--): track 0.00 -> 55.3 mm
- net Net-(U4A-+): track 0.00 -> 52.7 mm
- net Net-(D3-K): track 52.6 -> 0.00 mm, vias 2 -> 0
- net 9VOUT: track 0.00 -> 51.8 mm
- net Net-(IC1-L): track 0.00 -> 47.0 mm, vias 0 -> 1
- net Net-(D2-K): track 0.00 -> 44.2 mm
- net Net-(C20-Pad1): track 0.00 -> 42.6 mm, vias 0 -> 1
- net OUTPUT: track 0.00 -> 40.6 mm
- net Net-(U4A--): track 0.00 -> 37.8 mm
- net Net-(C1-Pad1): track 0.00 -> 37.6 mm
- net Net-(IC1-G): track 0.00 -> 30.5 mm
- net Net-(C4-Pad1): track 0.00 -> 29.1 mm
- net Earth: track 4.31 -> 29.0 mm, vias 2 -> 6
- net Net-(C17-Pad1): track 0.00 -> 23.9 mm, vias 0 -> 2
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- added copper zone on In1.Cu, net VREF
- removed copper zone on In1.Cu, net 9V

Commit message: finished pcb, commit before making wavy
Parts:
- J5: moved to F.Cu
- moved C20 7.29 mm to (152.8, 96.0)
- moved C17 6.90 mm to (128.0, 71.0), turned to 180 degrees
- moved C14 4.21 mm to (125.8, 77.8), turned to 180 degrees
- moved R18 3.20 mm to (153.8, 101.6)
- turned J5 to 90 degrees
Routing:
- net Net-(C20-Pad1): track 42.6 -> 58.7 mm
- net OUTPUT: track 40.6 -> 47.8 mm
- net Net-(C14-Pad2): track 4.28 -> 9.98 mm
- net Net-(U4A-+): track 52.7 -> 57.3 mm
- net Net-(IC1-G): track 30.5 -> 33.7 mm
- net Net-(C17-Pad1): track 23.9 -> 26.6 mm
- net CD-VCC: track 125.8 -> 126.7 mm
- net VREF: track 35.0 -> 34.2 mm

Commit message: pcb rev 1
Parts:
- added  : est-comic, cholm-footprints:est-comic, B.Cu at (117.4, 51.7)
- added R24: 1k, Resistor_SMD:R_1210_3225Metric, F.Cu at (152.0, 60.6)
- added R25: 3k, Resistor_SMD:R_1210_3225Metric, F.Cu at (152.0, 67.0)
- IC1: footprint Package_DIP:DIP-18_W7.62mm -> cholm-footprints:DIP794W45P254L1930H508Q16
- J12: value GND4 -> GND5
- moved IC1 9.74 mm to (130.9, 97.2)
- renumbered BASS1 to BASS, GAIN1 to GAIN, VOLUME1 to VOLUME
Connections:
- C2 pad 1: 9VOUT -> Net-(D2-A)
- D1 pad 1: 9VOUT -> Net-(D1-K)
- D2 pad 2: 9VOUT -> Net-(D2-A)
- U1 pad 8: 9VOUT -> Net-(D2-A)
Routing:
- net Net-(D2-A): track 0.00 -> 56.4 mm
- net 9VOUT: track 51.8 -> 0.00 mm
- net Net-(D1-K): track 0.00 -> 17.6 mm
- net Net-(BASS1-Pad3): track 24.4 -> 30.3 mm
- net Net-(U4A--): track 37.8 -> 41.8 mm
- net Net-(C16-Pad1): track 36.6 -> 40.5 mm
- net CD-VCC: track 126.7 -> 130.5 mm, vias 4 -> 5
- net Earth: track 29.0 -> 32.0 mm
- net Net-(IC1-L): track 47.0 -> 49.7 mm
- net Net-(U4B--): track 55.3 -> 53.5 mm
- net OUTPUT: track 47.8 -> 46.1 mm
- net Net-(IC1-F): track 49.8 -> 48.3 mm
- net Net-(C20-Pad1): track 58.7 -> 57.3 mm
- net Net-(C1-Pad1): track 37.6 -> 36.6 mm
- net VREF: track 34.2 -> 33.3 mm
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Other:
- board text added: "9V"
- board text added: "A MAN CANNOT KILL A GOD"
- board text added: "GND"
- board text added: "HELLERUNE OVERDRIVE REV 1.0 OFFWORLD SERPENT DEVICES"
- board text added: "IN"
- board text added: "LESS"
- board text added: "MORE"
- board text added: "OUT"
- board text added: "TO-SWITCH-2"

Commit message: pick and place files created
Parts:
- R4: footprint Resistor_SMD:R_MELF_MMB-0207 -> Resistor_SMD:R_MiniMELF_MMA-0204
- renumbered BASS to BASS1, GAIN to GAIN1, VOLUME to VOLUME1
Routing:
- net Net-(C16-Pad1): track 40.5 -> 41.1 mm
- net Net-(U4A--): track 41.8 -> 42.4 mm
Other:
- board text added: "."
