File: kicad/hellerune.kicad_sch (KiCad schematic)
At the start: 62 parts, among them IC1 CD4049UBE, J3 Conn_01x02_Female, J5 GND1, J6 9VOUT1, J6 9VOUT2, J6 GND2, J6 GND4, J7 GND3, J7 SWITCHY-2-B-IN-R1, J7 SWITCHY-2-B-IN-R2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

Commit message: updated schematic
Parts:
- removed U2: TL074, symbol Amplifier_Operational:TL074
- added C21: 10nF, Capacitors:0805, symbol Device:C_Small
- added J6: 9VOUT2, Connector_PinSocket_2.54mm:PinSocket_1x01_P2.54mm_Vertical, symbol Connector:Conn_01x01_Socket
- added J6: GND4, Connector_PinSocket_2.54mm:PinSocket_1x01_P2.54mm_Vertical, symbol Connector:Conn_01x01_Socket
- added U3, U4: TL072, symbol Amplifier_Operational:TL072
- BASS1, VOLUME1: symbol malice-striker-v2-rescue:R_POT_US-Device -> Device:R_Potentiometer_US
- C14: symbol fafnir-v1-rescue:CP1_Small-Device -> Device:C_Polarized_Small_US
- C15, C19, C2, C24, C25, C4, C6, C8: symbol malice-striker-v2-rescue:CP1_Small-Device -> Device:C_Polarized_Small_US
- GAIN1: symbol fafnir-v1-rescue:R_POT_US-Device -> Device:R_Potentiometer_US
- IC1: symbol fafnir-v1-rescue:CD4049UBE-CD4049UBE -> clholm-kicad-lib:CD4049UBE-CD4049UBE
- J3: symbol malice-striker-v2-rescue:Conn_01x02_Female-Connector -> Connector:Conn_01x02_Socket
- J5, J6, J7: symbol malice-striker-v2-rescue:Conn_01x01_Female-Connector -> Connector:Conn_01x01_Socket
- J6: value 9VOUT1 -> 9VIN; symbol malice-striker-v2-rescue:Conn_01x01_Female-Connector -> Connector:Conn_01x01_Socket
- J6: value 9VOUT2 -> 9VOUT1; symbol malice-striker-v2-rescue:Conn_01x01_Female-Connector -> Connector:Conn_01x01_Socket
Connections:
- net 9V: now also J6.1 (Pin_1), J6.1 (Pin_1), J6.1 (Pin_1)
- net 9VOUT: no longer J6.1 (Pin_1)
- net Earth: now also C21.2, J6.1 (Pin_1), U3.4 (V-), U4.4 (V-)
- net VREF: now also U3.5 (+), U4.5 (+)
- net at C23.1, R19.2: now also U3.6 (-)
- net at C24.1, R18.2, R20.1: now also U3.7
- net at R18.2, R18.2: now also U4.3 (+)
- net at C17.2, R19.1, R21.2: now also U4.2 (-)
- net at C13.1, C8.1, D3.1 (K)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: now also C21.1, U3.8 (V+), U4.8 (V+)
- net at C3.1, R3.1: now also U3.3 (+)
- net at C5.1, C7.2, R5.1: now also U3.1
- net at C5.2, R4.1, R5.2: now also U3.2 (-)
- net at R22.1, VOLUME1.3: now also U4.6 (-)
- net at C25.1, VOLUME1.1, VOLUME1.2: now also U4.7
- net at C17.1, C19.1, R21.1: now also U4.1
Other:
- moved on the sheet: C15, C17, C19, C25, J6, R15, R16, R18, R19, R21, R22, VOLUME1

Commit message: updated footprints
Parts:
- IC1: footprint DIP794W53P254L1930H508Q16N -> Package_DIP:DIP-18_W7.62mm
- R17: footprint (none) -> Resistor_SMD:R_2010_5025Metric
- R3: footprint Resistor_THT:R_Axial_DIN0414_L11.9mm_D4.5mm_P20.32mm_Horizontal -> Resistor_SMD:R_1210_3225Metric
- R4: footprint Resistor_THT:R_Axial_DIN0309_L9.0mm_D3.2mm_P15.24mm_Horizontal -> Resistor_SMD:R_MELF_MMB-0207
- R8: footprint (none) -> Resistor_SMD:R_0603_1608Metric
- U3, U4: footprint (none) -> Package_TO_SOT_SMD:TSOT-23-8
Changed lines of the file:
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@@
       (effects (font (size 1.27 1.27)))
     )
-    (property "Footprint" "" (at 173.99 144.78 0)
+    (property "Footprint" "Resistor_SMD:R_2010_5025Metric" (at 173.99 144.78 0)
       (effects (font (size 1.27 1.27)) hide)
     )
@@
       (effects (font (size 1.27 1.27)))
     )
-    (property "Footprint" "Resistor_THT:R_Axial_DIN0414_L11.9mm_D4.5mm_P20.32mm_Horizontal" (at 54.61 153.67 0)
+    (property "Footprint" "Resistor_SMD:R_1210_3225Metric" (at 54.61 153.67 0)
       (effects (font (size 1.27 1.27)) hide)
     )
@@
       (effects (font (size 1.27 1.27)))
     )
-    (property "Footprint" "" (at 215.9 55.88 0)
+    (property "Footprint" "Package_TO_SOT_SMD:TSOT-23-8" (at 215.9 55.88 0)
       (effects (font (size 1.27 1.27)) hide)
     )
@@
       (effects (font (size 1.27 1.27)))
     )
-    (property "Footprint" "" (at 254 53.34 0)
+    (property "Footprint" "Package_TO_SOT_SMD:TSOT-23-8" (at 254 53.34 0)
       (effects (font (size 1.27 1.27)) hide)
     )
@@
       (effects (font (size 1.27 1.27)))
     )
-    (property "Footprint" "" (at 137.16 160.02 0)
+    (property "Footprint" "Package_TO_SOT_SMD:TSOT-23-8" (at 137.16 160.02 0)
       (effects (font (size 1.27 1.27)) hide)
     )
@@
       (effects (font (size 1.27 1.27)) (justify left))
     )
-    (property "Footprint" "Resistor_THT:R_Axial_DIN0309_L9.0mm_D3.2mm_P15.24mm_Horizontal" (at 71.12 181.61 0)
+    (property "Footprint" "Resistor_SMD:R_MELF_MMB-0207" (at 71.12 181.61 0)
       (effects (font (size 1.27 1.27)) hide)
     )
@@
       (effects (font (size 1.27 1.27)) (justify left))
     )
-    (property "Footprint" "" (at 143.51 43.18 0)
+    (property "Footprint" "Package_TO_SOT_SMD:TSOT-23-8" (at 143.51 43.18 0)
       (effects (font (size 1.27 1.27)) hide)
     )
@@
       (effects (font (size 1.27 1.27)) (justify left))
     )
-    (property "Footprint" "" (at 121.92 43.18 0)
+    (property "Footprint" "Package_TO_SOT_SMD:TSOT-23-8" (at 121.92 43.18 0)
       (effects (font (size 1.27 1.27)) hide)
     )
@@
       (effects (font (size 1.27 1.27)))
     )
-    (property "Footprint" "DIP794W53P254L1930H508Q16N" (at 168.91 109.22 0)
+    (property "Footprint" "Package_DIP:DIP-18_W7.62mm" (at 168.91 109.22 0)
       (effects (font (size 1.27 1.27)) (justify left) hide)
     )
@@
       (effects (font (size 1.27 1.27)) (justify left))
     )
-    (property "Footprint" "" (at 105.41 114.3 0)
+    (property "Footprint" "Resistor_SMD:R_0603_1608Metric" (at 105.41 114.3 0)
       (effects (font (size 1.27 1.27)) hide)
     )
@@
       (effects (font (size 1.27 1.27)))
     )
-    (property "Footprint" "" (at 78.74 156.21 0)
-      (effects (font (size 1.27 1.27)) hide)
-    )
+    (property "Footprint" "Package_TO_SOT_SMD:TSOT-23-8" (at 78.74 156.21 0)
+      (effects (font (size 1.27 1.27)) hide)
+    )

Commit message: began PCB, traces
Parts:
- BASS1, GAIN1, VOLUME1: footprint clholm-kicad-lib:16MM_T.MOUNT -> cholm-footprints:16MM_T.MOUNT
- C1, C13, C21, C7: footprint Capacitors:0805 -> Capacitor_SMD:C_0805_2012Metric
- C11, C18: footprint (none) -> Capacitor_SMD:C_0402_1005Metric
- C12, C22, C3: footprint Capacitors:1206 -> Capacitor_SMD:C_1206_3216Metric
- C14: footprint (none) -> Capacitor_THT:CP_Radial_D5.0mm_P2.00mm
- C17: footprint Capacitors:0603 -> Capacitor_SMD:C_0603_1608Metric
- C2: footprint Capacitors:1206 -> Capacitor_THT:CP_Radial_D5.0mm_P2.00mm
- C23, C5: footprint Capacitors:0402 -> Capacitor_SMD:C_0402_1005Metric
- D1, D2, D3: value 1N5817 -> 1N4001; footprint Diode_SMD:D_SOD-123 -> Diode_SMD:D_SOD-323
- U3, U4: footprint Package_TO_SOT_SMD:TSOT-23-8 -> Package_SO:SOIC-8_3.9x4.9mm_P1.27mm
Changed lines of the file:
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@@
       (effects (font (size 1.27 1.27)) (justify left))
     )
-    (property "Footprint" "" (at 115.57 114.3 0)
+    (property "Footprint" "Capacitor_SMD:C_0402_1005Metric" (at 115.57 114.3 0)
       (effects (font (size 1.27 1.27)) hide)
     )
@@
       (effects (font (size 1.27 1.27)))
     )
-    (property "Footprint" "clholm-kicad-lib:16MM_T.MOUNT" (at 110.49 148.59 0)
+    (property "Footprint" "cholm-footprints:16MM_T.MOUNT" (at 110.49 148.59 0)
       (effects (font (size 1.27 1.27)) hide)
     )
@@
       (effects (font (size 1.27 1.27)))
     )
-    (property "Value" "1N5817" (at 30.48 32.3596 0)
-      (effects (font (size 1.27 1.27)))
-    )
-    (property "Footprint" "Diode_SMD:D_SOD-123" (at 30.48 31.115 0)
+    (property "Value" "1N4001" (at 30.48 32.3596 0)
+      (effects (font (size 1.27 1.27)))
+    )
+    (property "Footprint" "Diode_SMD:D_SOD-323" (at 30.48 31.115 0)
       (effects (font (size 1.27 1.27)) hide)
     )
@@
       (effects (font (size 1.27 1.27)) (justify left))
     )
-    (property "Footprint" "Capacitors:1206" (at 60.96 158.75 0)
+    (property "Footprint" "Capacitor_SMD:C_1206_3216Metric" (at 60.96 158.75 0)
       (effects (font (size 1.27 1.27)) hide)
     )
@@
       (effects (font (size 1.27 1.27)) (justify left))
     )
-    (property "Footprint" "Capacitors:0402" (at 110.49 167.64 0)
+    (property "Footprint" "Capacitor_SMD:C_0402_1005Metric" (at 110.49 167.64 0)
       (effects (font (size 1.27 1.27)) hide)
     )
@@
       (effects (font (size 1.27 1.27)))
     )
-    (property "Value" "1N5817" (at 99.06 32.3596 0)
-      (effects (font (size 1.27 1.27)))
-    )
-    (property "Footprint" "Diode_SMD:D_SOD-123" (at 99.06 31.115 0)
+    (property "Value" "1N4001" (at 99.06 32.3596 0)
+      (effects (font (size 1.27 1.27)))
+    )
+    (property "Footprint" "Diode_SMD:D_SOD-323" (at 99.06 31.115 0)
       (effects (font (size 1.27 1.27)) hide)
     )
@@
       (effects (font (size 1.27 1.27)) (justify left))
     )
-    (property "Footprint" "Capacitors:0805" (at 129.54 43.18 0)
+    (property "Footprint" "Capacitor_SMD:C_0805_2012Metric" (at 129.54 43.18 0)
       (effects (font (size 1.27 1.27)) hide)
     )
@@
       (effects (font (size 1.27 1.27)))
     )
-    (property "Footprint" "Package_TO_SOT_SMD:TSOT-23-8" (at 215.9 55.88 0)
+    (property "Footprint" "Package_SO:SOIC-8_3.9x4.9mm_P1.27mm" (at 215.9 55.88 0)
       (effects (font (size 1.27 1.27)) hide)
     )
@@
       (effects (font (size 1.27 1.27)))
     )
-    (property "Footprint" "Package_TO_SOT_SMD:TSOT-23-8" (at 254 53.34 0)
+    (property "Footprint" "Package_SO:SOIC-8_3.9x4.9mm_P1.27mm" (at 254 53.34 0)
       (effects (font (size 1.27 1.27)) hide)
     )
@@
       (effects (font (size 1.27 1.27)))
     )
-    (property "Footprint" "Capacitors:0603" (at 217.17 67.31 0)
+    (property "Footprint" "Capacitor_SMD:C_0603_1608Metric" (at 217.17 67.31 0)
       (effects (font (size 1.27 1.27)) hide)
     )
@@
       (effects (font (size 1.27 1.27)))
     )
-    (property "Footprint" "clholm-kicad-lib:16MM_T.MOUNT" (at 177.8 102.87 0)
+    (property "Footprint" "cholm-footprints:16MM_T.MOUNT" (at 177.8 102.87 0)
       (effects (font (size 1.27 1.27)) hide)
     )
@@
       (effects (font (size 1.27 1.27)))
     )
-    (property "Footprint" "Capacitors:0402" (at 80.01 167.64 0)
+    (property "Footprint" "Capacitor_SMD:C_0402_1005Metric" (at 80.01 167.64 0)
       (effects (font (size 1.27 1.27)) hide)
     )
@@
       (effects (font (size 1.27 1.27)) (justify left))
     )
-    (property "Footprint" "Capacitors:1206" (at 40.64 38.1 0)
+    (property "Footprint" "Capacitor_THT:CP_Radial_D5.0mm_P2.00mm" (at 40.64 38.1 0)
       (effects (font (size 1.27 1.27)) hide)
     )
@@
       (effects (font (size 1.27 1.27)) (justify left))
     )
-    (property "Footprint" "Capacitors:0805" (at 151.13 43.18 0)
+    (property "Footprint" "Capacitor_SMD:C_0805_2012Metric" (at 151.13 43.18 0)
       (effects (font (size 1.27 1.27)) hide)
     )
@@
       (effects (font (size 1.27 1.27)))
     )
-    (property "Footprint" "Package_TO_SOT_SMD:TSOT-23-8" (at 137.16 160.02 0)
+    (property "Footprint" "Package_SO:SOIC-8_3.9x4.9mm_P1.27mm" (at 137.16 160.02 0)
       (effects (font (size 1.27 1.27)) hide)
     )
@@
       (effects (font (size 1.27 1.27)) (justify right))
     )
-    (property "Footprint" "" (at 133.35 91.44 0)
+    (property "Footprint" "Capacitor_THT:CP_Radial_D5.0mm_P2.00mm" (at 133.35 91.44 0)
       (effects (font (size 1.27 1.27)) hide)
     )
@@
       (effects (font (size 1.27 1.27)) (justify left))
     )
-    (property "Footprint" "Package_TO_SOT_SMD:TSOT-23-8" (at 143.51 43.18 0)
+    (property "Footprint" "Package_SO:SOIC-8_3.9x4.9mm_P1.27mm" (at 143.51 43.18 0)
       (effects (font (size 1.27 1.27)) hide)
     )
@@
       (effects (font (size 1.27 1.27)) (justify left))
     )
-    (property "Footprint" "Capacitors:1206" (at 125.73 114.3 0)
+    (property "Footprint" "Capacitor_SMD:C_1206_3216Metric" (at 125.73 114.3 0)
       (effects (font (size 1.27 1.27)) hide)
     )
@@
       (effects (font (size 1.27 1.27)) (justify right))
     )
-    (property "Footprint" "clholm-kicad-lib:16MM_T.MOUNT" (at 251.46 64.77 0)
+    (property "Footprint" "cholm-footprints:16MM_T.MOUNT" (at 251.46 64.77 0)
       (effects (font (size 1.27 1.27)) hide)
     )
@@
       (effects (font (size 1.27 1.27)) (justify left))
     )
-    (property "Footprint" "Package_TO_SOT_SMD:TSOT-23-8" (at 121.92 43.18 0)
+    (property "Footprint" "Package_SO:SOIC-8_3.9x4.9mm_P1.27mm" (at 121.92 43.18 0)
       (effects (font (size 1.27 1.27)) hide)
     )
@@
       (effects (font (size 1.27 1.27)))
     )
-    (property "Footprint" "Capacitors:0805" (at 36.83 153.67 0)
+    (property "Footprint" "Capacitor_SMD:C_0805_2012Metric" (at 36.83 153.67 0)
       (effects (font (size 1.27 1.27)) hide)
     )
@@
       (effects (font (size 1.27 1.27)))
     )
-    (property "Footprint" "Capacitors:0805" (at 91.44 156.21 0)
+    (property "Footprint" "Capacitor_SMD:C_0805_2012Metric" (at 91.44 156.21 0)
       (effects (font (size 1.27 1.27)) hide)
     )
@@
       (effects (font (size 1.27 1.27)))
     )
-    (property "Footprint" "Capacitors:1206" (at 110.49 134.62 0)
+    (property "Footprint" "Capacitor_SMD:C_1206_3216Metric" (at 110.49 134.62 0)
       (effects (font (size 1.27 1.27)) hide)
     )
@@
       (effects (font (size 1.27 1.27)))
     )
-    (property "Footprint" "Package_TO_SOT_SMD:TSOT-23-8" (at 78.74 156.21 0)
+    (property "Footprint" "Package_SO:SOIC-8_3.9x4.9mm_P1.27mm" (at 78.74 156.21 0)
       (effects (font (size 1.27 1.27)) hide)
     )
@@
       (effects (font (size 1.27 1.27)))
     )
-    (property "Value" "1N5817" (at 69.85 20.9296 0)
-      (effects (font (size 1.27 1.27)))
-    )
-    (property "Footprint" "Diode_SMD:D_SOD-123" (at 69.85 19.685 0)
+    (property "Value" "1N4001" (at 69.85 20.9296 0)
+      (effects (font (size 1.27 1.27)))
+    )
+    (property "Footprint" "Diode_SMD:D_SOD-323" (at 69.85 19.685 0)
       (effects (font (size 1.27 1.27)) hide)
     )
@@
       (effects (font (size 1.27 1.27)))
     )
-    (property "Footprint" "" (at 191.77 114.3 0)
-      (effects (font (size 1.27 1.27)) hide)
-    )
+    (property "Footprint" "Capacitor_SMD:C_0402_1005Metric" (at 191.77 114.3 0)
+      (effects (font (size 1.27 1.27)) hide)
+    )

Commit message: pcb draft complete
Parts:
- added C22: 10nF, Capacitor_SMD:C_0805_2012Metric, symbol Device:C_Small
Connections:
- net Earth: now also C22.2
- net VREF: no longer IC1.1 (VCC), IC1.11 (E), IC1.5 (B), IC1.7 (C), IC1.9 (D)
- net CD-VCC: now reaches C13.1, C21.1, C8.1, D3.1 (K), R15.1, U3.8 (V+), U4.8 (V+)
- net CD-VCC: now also IC1.1 (VCC), IC1.11 (E), IC1.5 (B), IC1.7 (C), IC1.9 (D), C22.1
Other:
- moved on the sheet: C15, GAIN1, R15, R16

Commit message: pcb rev 1
Parts:
- added R24: 1k, Resistor_SMD:R_1210_3225Metric, symbol Device:R_Small_US
- added R25: 3k, Resistor_SMD:R_1210_3225Metric, symbol Device:R_Small_US
- IC1: footprint Package_DIP:DIP-18_W7.62mm -> cholm-footprints:DIP794W45P254L1930H508Q16
- J6: value GND4 -> GND5
Connections:
- net Earth: now also R25.1
- net 9VOUT: no longer names the net of C2.1, D2.2 (A), U1.8 (V+)
- net 9VOUT: now also R24.2, R25.2; no longer D1.1 (K)
- new net: D1.1 (K), R24.1
Other:
- moved on the sheet: D1
Changed lines of the file:
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@@
   (junction (at 38.1 77.47) (diameter 0) (color 0 0 0 0)
   )
-  (junction (at 50.8 35.56) (diameter 0) (color 0 0 0 0)
-  )
   (junction (at 119.38 35.56) (diameter 0) (color 0 0 0 0)
   )
@@
   (junction (at 177.8 102.87) (diameter 0) (color 0 0 0 0)
   )
+  (junction (at 30.48 35.56) (diameter 0) (color 0 0 0 0)
+  )
   (junction (at 162.56 35.56) (diameter 0) (color 0 0 0 0)
   )
@@
     (stroke (width 0) (type default))
   )
+  (wire (pts (xy 21.59 35.56) (xy 16.51 35.56))
+    (stroke (width 0) (type default))
+  )
   (wire (pts (xy 187.96 114.3) (xy 189.23 114.3))
     (stroke (width 0) (type default))
@@
     (stroke (width 0) (type default))
   )
-  (wire (pts (xy 50.8 35.56) (xy 50.8 40.64))
-    (stroke (width 0) (type default))
-  )
   (wire (pts (xy 173.99 102.87) (xy 173.99 99.06))
     (stroke (width 0) (type default))
@@
     (stroke (width 0) (type default))
   )
-  (wire (pts (xy 34.29 35.56) (xy 40.64 35.56))
+  (wire (pts (xy 26.67 35.56) (xy 30.48 35.56))
     (stroke (width 0) (type default))
   )
@@
     (stroke (width 0) (type default))
   )
-  (wire (pts (xy 40.64 35.56) (xy 50.8 35.56))
+  (wire (pts (xy 40.64 35.56) (xy 53.34 35.56))
     (stroke (width 0) (type default))
   )
@@
     (stroke (width 0) (type default))
   )
+  (wire (pts (xy 30.48 35.56) (xy 40.64 35.56))
+    (stroke (width 0) (type default))
+  )
   (wire (pts (xy 107.95 176.53) (xy 110.49 176.53))
     (stroke (width 0) (type default))
@@
     (stroke (width 0) (type default))
   )
+  (wire (pts (xy 16.51 35.56) (xy 16.51 30.48))
+    (stroke (width 0) (type default))
+  )
   (wire (pts (xy 241.3 55.88) (xy 241.3 64.77))
     (stroke (width 0) (type default))
@@
     (stroke (width 0) (type default))
   )
+  (wire (pts (xy 30.48 40.64) (xy 30.48 44.45))
+    (stroke (width 0) (type default))
+  )
   (wire (pts (xy 115.57 111.76) (xy 115.57 109.22))
     (stroke (width 0) (type default))
@@
     (stroke (width 0) (type default))
   )
-  (wire (pts (xy 22.86 35.56) (xy 26.67 35.56))
+  (wire (pts (xy 16.51 19.05) (xy 16.51 22.86))
     (stroke (width 0) (type default))
   )
@@
   )
   (wire (pts (xy 208.28 76.2) (xy 208.28 78.74))
-    (stroke (width 0) (type default))
-  )
-  (wire (pts (xy 50.8 35.56) (xy 53.34 35.56))
     (stroke (width 0) (type default))
   )
@@
     )
   )
-  (global_label "9V" (shape input) (at 22.86 35.56 180)
-    (effects (font (size 1.27 1.27)) (justify right))
-    (property "Intersheetrefs" "${INTERSHEET_REFS}" (at 22.86 35.56 0)
+  (global_label "9V" (shape input) (at 16.51 19.05 90)
+    (effects (font (size 1.27 1.27)) (justify left))
+    (property "Intersheetrefs" "${INTERSHEET_REFS}" (at 16.51 19.05 0)
       (effects (font (size 1.27 1.27)) hide)
     )
@@
     )
   )
-  (global_label "9VOUT" (shape input) (at 50.8 40.64 270)
-    (effects (font (size 1.27 1.27)) (justify right))
-    (property "Intersheetrefs" "${INTERSHEET_REFS}" (at 50.8 40.64 0)
-      (effects (font (size 1.27 1.27)) hide)
-    )
-  )
   (global_label "OUTPUT" (shape input) (at 273.05 53.34 0)
     (effects (font (size 1.27 1.27)) (justify left))
@@
         (path "/fed48d88-9175-44c3-9445-f07dec3c93d4"
           (reference "#PWR0102") (unit 1)
+        )
+      )
+    )
+  )
+  (symbol (lib_id "Device:R_Small_US") (at 24.13 35.56 90) (unit 1)
+    (in_bom yes) (on_board yes) (dnp no)
+    (property "Reference" "R24" (at 24.13 40.64 90)
+      (effects (font (size 1.27 1.27)))
+    )
+    (property "Value" "1k" (at 24.13 38.1 90)
+      (effects (font (size 1.27 1.27)))
+    )
+    (property "Footprint" "Resistor_SMD:R_1210_3225Metric" (at 24.13 35.56 0)
+      (effects (font (size 1.27 1.27)) hide)
+    )
+    (property "Datasheet" "~" (at 24.13 35.56 0)
+      (effects (font (size 1.27 1.27)) hide)
+    )
+    (pin "1")
+    (pin "2")
+    (instances
+      (project "hellerune"
+        (path "/7036af83-ac22-4511-9ae8-fe6718cb4d9e"
+          (reference "R24") (unit 1)
+        )
+      )
+      (project "malice-striker-v2"
+        (path "/fed48d88-9175-44c3-9445-f07dec3c93d4"
+          (reference "R14") (unit 1)
         )
       )
@@
     )
   )
-  (symbol (lib_id "Diode:1N5817") (at 30.48 35.56 180) (unit 1)
-    (in_bom yes) (on_board yes) (dnp no)
-    (property "Reference" "D1" (at 30.48 30.0482 0)
-      (effects (font (size 1.27 1.27)))
-    )
-    (property "Value" "1N4001" (at 30.48 32.3596 0)
-      (effects (font (size 1.27 1.27)))
-    )
-    (property "Footprint" "Diode_SMD:D_SOD-323" (at 30.48 31.115 0)
-      (effects (font (size 1.27 1.27)) hide)
-    )
-    (property "Datasheet" "http://www.vishay.com/docs/88525/1n5817.pdf" (at 30.48 35.56 0)
+  (symbol (lib_id "power:Earth") (at 30.48 44.45 0) (unit 1)
+    (in_bom yes) (on_board yes) (dnp no)
+    (property "Reference" "#PWR022" (at 30.48 50.8 0)
+      (effects (font (size 1.27 1.27)) hide)
+    )
+    (property "Value" "Earth" (at 30.48 48.26 0)
+      (effects (font (size 1.27 1.27)) hide)
+    )
+    (property "Footprint" "" (at 30.48 44.45 0)
+      (effects (font (size 1.27 1.27)) hide)
+    )
+    (property "Datasheet" "~" (at 30.48 44.45 0)
+      (effects (font (size 1.27 1.27)) hide)
+    )
+    (pin "1")
+    (instances
+      (project "hellerune"
+        (path "/7036af83-ac22-4511-9ae8-fe6718cb4d9e"
+          (reference "#PWR022") (unit 1)
+        )
+      )
+      (project "malice-striker-v2"
+        (path "/fed48d88-9175-44c3-9445-f07dec3c93d4"
+          (reference "#PWR01") (unit 1)
+        )
+      )
+    )
+  )
+  (symbol (lib_id "Diode:1N5817") (at 16.51 26.67 90) (unit 1)
+    (in_bom yes) (on_board yes) (dnp no)
+    (property "Reference" "D1" (at 22.0218 26.67 0)
+      (effects (font (size 1.27 1.27)))
+    )
+    (property "Value" "1N4001" (at 19.7104 26.67 0)
+      (effects (font (size 1.27 1.27)))
+    )
+    (property "Footprint" "Diode_SMD:D_SOD-323" (at 20.955 26.67 0)
+      (effects (font (size 1.27 1.27)) hide)
+    )
+    (property "Datasheet" "http://www.vishay.com/docs/88525/1n5817.pdf" (at 16.51 26.67 0)
       (effects (font (size 1.27 1.27)) hide)
     )
@@
       (effects (font (size 1.27 1.27)) (justify left))
     )
-    (property "Value" "GND4" (at 43.8912 89.281 0)
+    (property "Value" "GND5" (at 43.8912 89.281 0)
       (effects (font (size 1.27 1.27)) (justify left))
     )
@@
     )
   )
+  (symbol (lib_id "Device:R_Small_US") (at 30.48 38.1 180) (unit 1)
+    (in_bom yes) (on_board yes) (dnp no)
+    (property "Reference" "R25" (at 35.56 38.1 90)
+      (effects (font (size 1.27 1.27)))
+    )
+    (property "Value" "3k" (at 33.02 38.1 90)
+      (effects (font (size 1.27 1.27)))
+    )
+    (property "Footprint" "Resistor_SMD:R_1210_3225Metric" (at 30.48 38.1 0)
+      (effects (font (size 1.27 1.27)) hide)
+    )
+    (property "Datasheet" "~" (at 30.48 38.1 0)
+      (effects (font (size 1.27 1.27)) hide)
+    )
+    (pin "1")
+    (pin "2")
+    (instances
+      (project "hellerune"
+        (path "/7036af83-ac22-4511-9ae8-fe6718cb4d9e"
+          (reference "R25") (unit 1)
+        )
+      )
+      (project "malice-striker-v2"
+        (path "/fed48d88-9175-44c3-9445-f07dec3c93d4"
+          (reference "R14") (unit 1)
+        )
+      )
+    )
+  )
   (symbol (lib_id "Device:C_Polarized_Small_US") (at 107.95 43.18 0) (unit 1)
     (in_bom yes) (on_board yes) (dnp no)
@@
       (effects (font (size 1.27 1.27)))
     )
-    (property "Footprint" "Package_DIP:DIP-18_W7.62mm" (at 168.91 109.22 0)
+    (property "Footprint" "cholm-footprints:DIP794W45P254L1930H508Q16" (at 168.91 109.22 0)
       (effects (font (size 1.27 1.27)) (justify left) hide)
     )

Commit message: pick and place files created
Parts:
- R4: footprint Resistor_SMD:R_MELF_MMB-0207 -> Resistor_SMD:R_MiniMELF_MMA-0204
Changed lines of the file:
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@@
       (effects (font (size 1.27 1.27)) (justify left))
     )
-    (property "Footprint" "Resistor_SMD:R_MELF_MMB-0207" (at 71.12 181.61 0)
+    (property "Footprint" "Resistor_SMD:R_MiniMELF_MMA-0204" (at 71.12 181.61 0)
       (effects (font (size 1.27 1.27)) hide)
     )
