File: kicad/hellerune-switchy.kicad_pcb (KiCad board)
At the start: 2 copper layers, 20.2 x 16.2 mm, 4 parts, among them J1 LED CONNECT, J2 BOARD CONNECTIONS

Commit message: gerber files for the second switch breakout board
Other:
- board text added: "CLR"
